File: FlatSatHub.kicad_pcb (KiCad board)
At the start: 4 copper layers, 166.3 x 166.3 mm, 34 parts, among them J1 Jack-DC, J10 DB26_Male_HighDensity_Mountin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, J11 Conn_02x02_Odd_Even, J12 DB26_Male_HighDensity_Mountin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, J13 Conn_02x02_Odd_Even, J14 DB26_Male_HighDensity_Mountin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, J15 Conn_02x02_Odd_Even, J16 DB26_Male_HighDensity_Mountin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, J17 Conn_02x02_Odd_Even, J2 DB26_Male_HighDensity_Mountin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, J3 Conn_02x02_Odd_Even, J4 DB26_Male_HighDensity_Mountin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, J5 Conn_02x02_Odd_Even, J6 DB26_Male_HighDensity_Mountin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, J7 Conn_02x02_Odd_Even, J8 DB26_Male_HighDensity_Mountin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, J9 Conn_02x02_Odd_Even, SW1 SW_SPDT, SW10 SW_SPDT, SW11 SW_SPDT, SW2 SW_DIP_x03, SW3 SW_DIP_x03, SW4 SW_DIP_x03, SW5 SW_DIP_x03, SW6 SW_DIP_x03, SW7 SW_DIP_x03, SW8 SW_DIP_x03, SW9 SW_DIP_x03

Commit message: minor improvements
Parts:
- removed SW11: SW_SPDT, Button_Switch_SMD:SW_SPDT_PCM12
- added D1: GREEN LED, LED_SMD:LED_0603_1608Metric_Pad1.05x0.95mm_HandSolder, F.Cu at (108.1, 89.8)
- added D2: GREEN LED, LED_SMD:LED_0603_1608Metric_Pad1.05x0.95mm_HandSolder, F.Cu at (121.4, 89.6)
- added D3: GREEN_LED, LED_SMD:LED_0603_1608Metric_Pad1.05x0.95mm_HandSolder, F.Cu at (120.2, 108.6)
- added R1: R, Resistor_SMD:R_0603_1608Metric_Pad1.05x0.95mm_HandSolder, F.Cu at (108.1, 84.7)
- added R2: R, Resistor_SMD:R_0603_1608Metric_Pad1.05x0.95mm_HandSolder, F.Cu at (121.4, 84.5)
- added R3: R, Resistor_SMD:R_0603_1608Metric_Pad1.05x0.95mm_HandSolder, F.Cu at (120.2, 103.6)
- SW1: value SW_SPDT -> SW_DIP_x02; footprint Button_Switch_SMD:SW_SPDT_PCM12 -> Button_Switch_THT:SW_DIP_SPSTx02_Slide_6.7x6.64mm_W7.62mm_P2.54mm_LowProfile
- SW10: value SW_SPDT -> SW_SPST; footprint Button_Switch_SMD:SW_SPDT_PCM12 -> Button_Switch_THT:SW_DIP_SPSTx01_Slide_9.78x4.72mm_W7.62mm_P2.54mm
- moved SW1 11.8 mm to (113.2, 93.4)
- moved SW10 10.4 mm to (114.4, 112.4)
- moved C2 6.98 mm to (99.2, 99.7)
- moved C1 1.42 mm to (80.2, 94.7)
- moved J1 0.58 mm to (165.0, 130.7), turned to 67.5 degrees
Connections:
- SW1 pad 1: Vbat -> GND
- SW1 pad 2: /Vin -> GND
- SW1 pad 3: Net-(SW1-Pad3) -> Net-(C1-Pad11)
- SW10 pad 1: Net-(SW10-Pad1) -> /Vin
- SW10 pad 2: GND -> Vbat

Commit message: route and add documentation for schematic
Parts:
- turned R1 to 270 degrees
- turned R2 to 270 degrees
- turned R3 to 270 degrees
Routing:
- net /I2C1_SCL: track 0.00 -> 565.4 mm, vias 0 -> 11
- net /I2C1_SDA: track 0.00 -> 523.1 mm, vias 0 -> 8
- net /SPI1_SCK: track 0.00 -> 522.1 mm, vias 0 -> 8
- net /I2C2_SDA: track 0.00 -> 509.5 mm, vias 0 -> 8
- net /SPI1_MOSI: track 0.00 -> 503.3 mm, vias 0 -> 8
- net /I2C2_SCL: track 0.00 -> 500.3 mm, vias 0 -> 7
- net /CAN1_RX: track 0.00 -> 493.1 mm, vias 0 -> 5
- net /SPI4_SCK: track 0.00 -> 489.1 mm, vias 0 -> 8
- net /SPI1_MISO: track 0.00 -> 488.7 mm, vias 0 -> 8
- net /SPI4_MISO: track 0.00 -> 488.6 mm, vias 0 -> 7
- net /SPI4_MOSI: track 0.00 -> 482.7 mm
- net /SPI1_SS: track 0.00 -> 481.4 mm, vias 0 -> 7
- net /SPI4_SS: track 0.00 -> 474.1 mm, vias 0 -> 7
- net /CAN1_TX: track 0.00 -> 470.8 mm, vias 0 -> 4
- net /Vin: track 0.00 -> 150.0 mm, vias 0 -> 3
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- added copper zone on In1.Cu, net Vbat
- removed copper zone on In1.Cu, net VCC

Commit message: add markings for switchs
Routing:
- net GND: track 0.00 -> 112.4 mm, vias 0 -> 1
- net 3V3: track 0.00 -> 48.7 mm, vias 0 -> 1
Other:
- board text added: "3V3"
- board text added: "5V"
- board text added: "Vbat"
