File: FlatSatHub.kicad_pcb (KiCad board)
At the start: 4 copper layers, 166.3 x 166.3 mm, 38 parts, among them J1 Jack-DC, J10 DB26_Male_HighDensity_Mountin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, J11 HEADER_4x2, J12 DB26_Male_HighDensity_Mountin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, J13 HEADER_4x2, J14 DB26_Male_HighDensity_Mountin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, J15 DB26_Male_HighDensity_Mountin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, J16 DB26_Male_HighDensity_Mountin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, J2 HEADER_4x2, J3 HEADER_4x2, J4 DB26_Male_HighDensity_Mountin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, J5 HEADER_4x2, J6 DB26_Male_HighDensity_Mountin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, J7 HEADER_4x2, J8 DB26_Male_HighDensity_Mountin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, J9 HEADER_4x2, SW1 SW_DIP_x02, SW10 SW_SPST, SW2 SW_DIP_x03, SW3 SW_DIP_x03, SW4 SW_DIP_x03, SW5 SW_DIP_x03, SW6 SW_DIP_x03, SW7 SW_DIP_x03, SW8 SW_DIP_x03, SW9 SW_DIP_x03

Commit message: New layout with FPGA
- Added FPGA to ease UART and SPI signals routing
- Cleaned layout using start and circle patterns for remaining signals
- Replaced DCDC modules with better TI components

Missing stuff:
- per module PSU switch
- spare FPGA IOs connector?
- silk screen
- ...

Signed-off-by: Alexis Jeandet <alexis.jeandet@member.fsf.org>
Parts:
- removed J11, J13, J2, J3, J7, J9: HEADER_4x2, Connector_PinHeader_2.54mm:PinHeader_2x04_P2.54mm_Vertical
- removed J15: DB26_Male_HighDensity_MountingHoles, Connector_Dsub:DSUB-26-HD_Female_Horizontal_P2.29x1.98mm_EdgePinOffset3.03mm_Housed_MountingHolesOffset4.94mm
- removed SW1: SW_DIP_x02, Button_Switch_THT:SW_DIP_SPSTx02_Slide_6.7x6.64mm_W7.62mm_P2.54mm_LowProfile
- removed SW2, SW3, SW4, SW5, SW6, SW7, SW8, SW9: SW_DIP_x03, Button_Switch_THT:SW_DIP_SPSTx03_Slide_9.78x9.8mm_W7.62mm_P2.54mm
- added C10: 47u, Capacitor_SMD:C_1210_3225Metric_Pad1.42x2.65mm_HandSolder, B.Cu at (125.6, 158.0)
- added C11: 2.2uF, Capacitor_SMD:C_1210_3225Metric_Pad1.42x2.65mm_HandSolder, B.Cu at (172.6, 72.5)
- added C12: 2.2uF, Capacitor_SMD:C_1210_3225Metric_Pad1.42x2.65mm_HandSolder, B.Cu at (169.3, 72.5)
- added C13: 2.2uF, Capacitor_SMD:C_1210_3225Metric_Pad1.42x2.65mm_HandSolder, F.Cu at (169.3, 72.5)
- added C14: 2.2uF, Capacitor_SMD:C_1210_3225Metric_Pad1.42x2.65mm_HandSolder, F.Cu at (172.6, 72.5)
- added C15: C, Capacitor_SMD:C_0603_1608Metric_Pad1.05x0.95mm_HandSolder, F.Cu at (164.0, 73.6)
- added C16: C, Capacitor_SMD:C_0603_1608Metric_Pad1.05x0.95mm_HandSolder, F.Cu at (156.9, 70.5)
- added C17: C, Capacitor_SMD:C_0603_1608Metric_Pad1.05x0.95mm_HandSolder, F.Cu at (159.4, 69.7)
- added C18: 47u, Capacitor_SMD:C_1210_3225Metric_Pad1.42x2.65mm_HandSolder, B.Cu at (151.8, 74.1)
- added C19: 47u, Capacitor_SMD:C_1210_3225Metric_Pad1.42x2.65mm_HandSolder, B.Cu at (151.8, 67.5)
- added C20: 47u, Capacitor_SMD:C_1210_3225Metric_Pad1.42x2.65mm_HandSolder, B.Cu at (151.8, 70.8)
- added C21: 100nF, Capacitor_SMD:C_0402_1005Metric, B.Cu at (103.1, 102.4)
- added C22: 100nF, Capacitor_SMD:C_0402_1005Metric, B.Cu at (90.5, 110.1)
- added C23: 100nF, Capacitor_SMD:C_0402_1005Metric, B.Cu at (96.0, 110.1)
- added C24: 100nF, Capacitor_SMD:C_0402_1005Metric, B.Cu at (75.5, 117.1)
- added C25: 100nF, Capacitor_SMD:C_0402_1005Metric, B.Cu at (86.2, 95.4)
- added C26: 100nF, Capacitor_SMD:C_0402_1005Metric, B.Cu at (103.1, 96.9)
- added C27: 100nF, Capacitor_SMD:C_0402_1005Metric, B.Cu at (93.4, 100.9)
- added C28: 100nF, Capacitor_SMD:C_0402_1005Metric, B.Cu at (92.5, 93.2)
- added C29: 100nF, Capacitor_SMD:C_0402_1005Metric, B.Cu at (86.3, 107.4)
- added C3: 2.2uF, Capacitor_SMD:C_1210_3225Metric_Pad1.42x2.65mm_HandSolder, F.Cu at (123.8, 175.6)
- added C30: 100nF, Capacitor_SMD:C_0402_1005Metric, F.Cu at (104.9, 112.5)
- added C31: 100nF, Capacitor_SMD:C_0402_1005Metric, B.Cu at (91.5, 93.2)
- added C32: 100nF, Capacitor_SMD:C_0402_1005Metric, B.Cu at (93.3, 116.5)
- added C33: 100nF, Capacitor_SMD:C_0402_1005Metric, B.Cu at (96.5, 93.2)
- added C34: 100nF, Capacitor_SMD:C_0402_1005Metric, F.Cu at (105.6, 91.5)
- added C35: 100nF, Capacitor_SMD:C_0402_1005Metric, B.Cu at (86.3, 105.9)
- added C36: 100nF, Capacitor_SMD:C_0402_1005Metric, B.Cu at (102.5, 93.2)
- added C37: 100nF, Capacitor_SMD:C_0402_1005Metric, B.Cu at (93.0, 110.1)
- added C38: 100nF, Capacitor_SMD:C_0402_1005Metric, B.Cu at (95.0, 93.2)
- added C39: 100nF, Capacitor_SMD:C_0402_1005Metric, B.Cu at (103.1, 100.9)
- added C4: 2.2uF, Capacitor_SMD:C_1210_3225Metric_Pad1.42x2.65mm_HandSolder, F.Cu at (123.8, 178.9)
- added C40: 100nF, Capacitor_SMD:C_0402_1005Metric, B.Cu at (87.5, 110.1)
- added C41: 100nF, Capacitor_SMD:C_0402_1005Metric, F.Cu at (84.0, 111.8)
- added C42: 100nF, Capacitor_SMD:C_0402_1005Metric, B.Cu at (94.5, 110.1)
- added C43: 10uF, Capacitor_SMD:C_1206_3216Metric_Pad1.42x1.75mm_HandSolder, F.Cu at (119.1, 107.2)
- added C44: 10uF, Capacitor_SMD:C_1206_3216Metric_Pad1.42x1.75mm_HandSolder, B.Cu at (117.2, 93.5)
- added C45: 10uF, Capacitor_SMD:C_1206_3216Metric_Pad1.42x1.75mm_HandSolder, B.Cu at (110.8, 93.5)
- added C46: 10uF, Capacitor_SMD:C_1206_3216Metric_Pad1.42x1.75mm_HandSolder, B.Cu at (115.0, 108.7)
- added C47: 10uF, Capacitor_SMD:C_1206_3216Metric_Pad1.42x1.75mm_HandSolder, B.Cu at (115.3, 102.1)
- added C48: 2.2uF, Capacitor_SMD:C_1210_3225Metric_Pad1.42x2.65mm_HandSolder, B.Cu at (144.0, 108.5)
- added C49: 2.2uF, Capacitor_SMD:C_1210_3225Metric_Pad1.42x2.65mm_HandSolder, B.Cu at (140.7, 108.5)
- added C5: C, Capacitor_SMD:C_0603_1608Metric_Pad1.05x0.95mm_HandSolder, F.Cu at (122.8, 170.2)
- added C50: 2.2uF, Capacitor_SMD:C_1210_3225Metric_Pad1.42x2.65mm_HandSolder, F.Cu at (140.7, 108.5)
- added C51: 2.2uF, Capacitor_SMD:C_1210_3225Metric_Pad1.42x2.65mm_HandSolder, F.Cu at (144.0, 108.5)
- added C52: C, Capacitor_SMD:C_0603_1608Metric_Pad1.05x0.95mm_HandSolder, F.Cu at (135.3, 109.5)
- added C53: C, Capacitor_SMD:C_0603_1608Metric_Pad1.05x0.95mm_HandSolder, F.Cu at (128.2, 106.5)
- added C54: C, Capacitor_SMD:C_0603_1608Metric_Pad1.05x0.95mm_HandSolder, F.Cu at (130.8, 105.7)
- added C55: 47u, Capacitor_SMD:C_1210_3225Metric_Pad1.42x2.65mm_HandSolder, B.Cu at (123.1, 110.0)
- added C56: 47u, Capacitor_SMD:C_1210_3225Metric_Pad1.42x2.65mm_HandSolder, B.Cu at (123.1, 103.4)
- added C57: 47u, Capacitor_SMD:C_1210_3225Metric_Pad1.42x2.65mm_HandSolder, B.Cu at (123.1, 106.7)
- added C6: C, Capacitor_SMD:C_0603_1608Metric_Pad1.05x0.95mm_HandSolder, F.Cu at (125.8, 163.1)
- added C7: C, Capacitor_SMD:C_0603_1608Metric_Pad1.05x0.95mm_HandSolder, F.Cu at (126.6, 165.7)
- added C8: 47u, Capacitor_SMD:C_1210_3225Metric_Pad1.42x2.65mm_HandSolder, B.Cu at (122.3, 158.0)
- added C9: 47u, Capacitor_SMD:C_1210_3225Metric_Pad1.42x2.65mm_HandSolder, B.Cu at (128.9, 158.0)
- added D4: LED, Resistor_SMD:R_0603_1608Metric_Pad1.05x0.95mm_HandSolder, F.Cu at (77.0, 114.1)
- added D5: D_Schottky, Diode_SMD:D_SMC_Handsoldering, F.Cu at (126.4, 112.1)
- added DONE1: LED, Resistor_SMD:R_0603_1608Metric_Pad1.05x0.95mm_HandSolder, F.Cu at (100.6, 115.3)
- added J17: Conn_01x06, Connector_PinHeader_2.54mm:PinHeader_1x06_P2.54mm_Vertical, F.Cu at (104.0, 126.7)
- added L1: 7.2uH, Inductor_SMD:L_Wuerth_HCI-1040, B.Cu at (124.3, 165.9)
- added L2: 7.2uH, Inductor_SMD:L_Wuerth_HCI-1040, B.Cu at (159.6, 72.0)
- added L3: 2.2uH, Inductor_SMD:L_1206_3216Metric_Pad1.42x1.75mm_HandSolder, F.Cu at (115.3, 102.1)
- added L4: 2.2uH, Inductor_SMD:L_1206_3216Metric_Pad1.42x1.75mm_HandSolder, F.Cu at (115.0, 108.7)
- added L5: 7.2uH, Inductor_SMD:L_Wuerth_HCI-1040, B.Cu at (131.0, 108.0)
- added R10: R, Resistor_SMD:R_0603_1608Metric_Pad1.05x0.95mm_HandSolder, F.Cu at (156.9, 69.0)
- added R11: R, Resistor_SMD:R_0603_1608Metric_Pad1.05x0.95mm_HandSolder, F.Cu at (158.6, 66.4)
- added R12: R, Resistor_SMD:R_0603_1608Metric_Pad1.05x0.95mm_HandSolder, F.Cu at (162.2, 66.4)
- added R13: 2K2, Resistor_SMD:R_0402_1005Metric, F.Cu at (73.9, 112.6)
- added R14: 2K2, Resistor_SMD:R_0402_1005Metric, B.Cu at (75.5, 116.1)
- added R15: 10k, Resistor_SMD:R_0402_1005Metric, F.Cu at (102.0, 124.1)
- added R16: 2K2, Resistor_SMD:R_0402_1005Metric, F.Cu at (73.9, 114.1)
- added R17: 2K2, Resistor_SMD:R_0402_1005Metric, B.Cu at (101.8, 115.1)
- added R18: 10k, Resistor_SMD:R_0402_1005Metric, B.Cu at (91.1, 103.3)
- added R19: 10k, Resistor_SMD:R_0402_1005Metric, B.Cu at (102.0, 105.6)
- added R20: 10k, Resistor_SMD:R_0402_1005Metric, F.Cu at (103.3, 114.6)
- added R21: 10k, Resistor_SMD:R_0402_1005Metric, F.Cu at (102.3, 114.6)
- added R22: R, Resistor_SMD:R_0603_1608Metric_Pad1.05x0.95mm_HandSolder, F.Cu at (140.9, 105.2)
- added R23: R, Resistor_SMD:R_0603_1608Metric_Pad1.05x0.95mm_HandSolder, F.Cu at (140.9, 103.7)
- added R24: R, Resistor_SMD:R_0603_1608Metric_Pad1.05x0.95mm_HandSolder, F.Cu at (137.1, 102.4)
- added R25: R, Resistor_SMD:R_0603_1608Metric_Pad1.05x0.95mm_HandSolder, F.Cu at (128.2, 104.9)
- added R26: R, Resistor_SMD:R_0603_1608Metric_Pad1.05x0.95mm_HandSolder, F.Cu at (130.0, 102.4)
- added R27: R, Resistor_SMD:R_0603_1608Metric_Pad1.05x0.95mm_HandSolder, F.Cu at (133.5, 102.4)
- added R4: R, Resistor_SMD:R_0603_1608Metric_Pad1.05x0.95mm_HandSolder, F.Cu at (127.3, 163.1)
- added R5: R, Resistor_SMD:R_0603_1608Metric_Pad1.05x0.95mm_HandSolder, F.Cu at (129.9, 164.9)
- added R6: R, Resistor_SMD:R_0603_1608Metric_Pad1.05x0.95mm_HandSolder, F.Cu at (129.9, 168.4)
- added R7: R, Resistor_SMD:R_0603_1608Metric_Pad1.05x0.95mm_HandSolder, F.Cu at (169.6, 69.2)
- added R8: R, Resistor_SMD:R_0603_1608Metric_Pad1.05x0.95mm_HandSolder, F.Cu at (169.6, 67.7)
- added R9: R, Resistor_SMD:R_0603_1608Metric_Pad1.05x0.95mm_HandSolder, F.Cu at (165.7, 66.4)
- added SW11: SW_Push, Button_Switch_SMD:SW_SPST_EVQPE1, F.Cu at (75.3, 117.1)
- added U1: TPS54560B, Package_SO:Texas_R-PDSO-G8_EP2.95x4.9mm_Mask2.4x3.1mm, F.Cu at (126.3, 170.2)
- added U2: TPS54560B, Package_SO:Texas_R-PDSO-G8_EP2.95x4.9mm_Mask2.4x3.1mm, F.Cu at (164.0, 70.0)
- added U3: ASDMB-xxxMHz, Oscillator:Oscillator_SMD_Abracon_ASDMB-4Pin_2.5x2.0mm, B.Cu at (91.3, 116.1)
- added U4: ICE40HX1K-4K-TQ144, Package_QFP:TQFP-144_20x20mm_P0.5mm, F.Cu at (94.8, 101.7)
- added U5: M25PX32-VMW, Package_SO:SOIJ-8_5.3x5.3mm_P1.27mm, B.Cu at (96.6, 104.4)
- added U6: tps6240x, Package_SON:Texas_S-PVSON-N10_ThermalVias, F.Cu at (115.1, 105.4)
- added U7: TLV73325PDBV, Package_TO_SOT_SMD:SOT-23-5, B.Cu at (113.9, 93.0)
- added U8: TPS54560B, Package_SO:Texas_R-PDSO-G8_EP2.95x4.9mm_Mask2.4x3.1mm, F.Cu at (135.3, 106.0)
- C1: value CINCON-SIPSMT10-12 -> 2.2uF; footprint FlatSatHub:CINCON-SIPSMT10-12 -> Capacitor_SMD:C_1210_3225Metric_Pad1.42x2.65mm_HandSolder; moved to B.Cu
- C2: value bel-xRBA-06E2Ax -> 2.2uF; footprint FlatSatHub:BEL-xRBA-06E2Ax -> Capacitor_SMD:C_1210_3225Metric_Pad1.42x2.65mm_HandSolder; moved to B.Cu
- D1, D2: value LED -> D_Schottky; footprint LED_SMD:LED_0603_1608Metric_Pad1.05x0.95mm_HandSolder -> Diode_SMD:D_SMC_Handsoldering
- D3: footprint LED_SMD:LED_0603_1608Metric_Pad1.05x0.95mm_HandSolder -> Resistor_SMD:R_0603_1608Metric_Pad1.05x0.95mm_HandSolder
- J5: value HEADER_4x2 -> DB26_Male_HighDensity_MountingHoles; footprint Connector_PinHeader_2.54mm:PinHeader_2x04_P2.54mm_Vertical -> Connector_Dsub:DSUB-26-HD_Female_Horizontal_P2.29x1.98mm_EdgePinOffset3.03mm_Housed_MountingHolesOffset4.94mm
- SW10: value SW_SPST -> SW_DIP_x02; footprint Button_Switch_THT:SW_DIP_SPSTx01_Slide_9.78x4.72mm_W7.62mm_P2.54mm -> Button_Switch_THT:SW_DIP_SPSTx02_Slide_9.78x7.26mm_W7.62mm_P2.54mm
- moved J5 128.7 mm to (170.2, 92.4), turned to 90 degrees
- moved C1 94.8 mm to (123.8, 178.9), turned to 180 degrees
- moved R1 93.0 mm to (127.1, 175.8), turned to 90 degrees
- moved R2 91.6 mm to (128.6, 175.8)
- moved C2 79.7 mm to (123.8, 175.6), turned to 180 degrees
- moved D1 72.5 mm to (120.2, 161.3), turned to 90 degrees
- moved R3 69.1 mm to (129.9, 172.0), turned to 90 degrees
- moved D3 43.4 mm to (77.0, 112.6), turned to 180 degrees
- moved SW10 41.4 mm to (153.0, 127.3), turned to 157 degrees
- moved D2 36.3 mm to (155.1, 76.1), turned to 180 degrees
Connections:
- C1 pad 1: 3V3 -> /Sheet5F4EF57F/VBAT
- C1 pad 2: 3V3 -> GND
- C2 pad 1: 5V -> /Sheet5F4EF57F/VBAT
- C2 pad 2: Net-(C2-Pad2) -> GND
- D1 pad 1: Net-(D1-Pad1) -> Net-(C5-Pad1)
- D1 pad 2: Net-(C2-Pad6) -> GND
- D2 pad 1: Net-(D2-Pad1) -> Net-(C15-Pad1)
- D2 pad 2: Net-(C1-Pad11) -> GND
- D3 pad 1: Net-(D3-Pad1) -> /Sheet5F604EE5/LED1
- D3 pad 2: Vbat -> Net-(D3-Pad2)
- J1 pad 1: /Vin -> /Sheet5F4EF57F/VBAT
- J10 pad 12: /SPI1_MOSI -> /MOD4_SPI1_MOSI
- J10 pad 13: /SPI4_MISO -> /MOD4_SPI2_MISO
- J10 pad 15: /sheet5F23178F/UART1_TX -> /MOD4_UART1_TX
- J10 pad 16: Net-(J10-Pad16) -> (no net)
- J10 pad 17: Net-(J10-Pad17) -> (no net)
- J10 pad 2: /SPI1_MISO -> /MOD4_SPI1_MISO
- J10 pad 22: /SPI4_MOSI -> /MOD4_SPI2_MOSI
- J10 pad 23: /sheet5F23178F/UART1_RX -> /MOD4_UART1_RX
- J10 pad 24: /sheet5F23178F/UART2_TX -> /MOD4_UART2_TX
- J10 pad 25: Net-(J10-Pad25) -> (no net)
- J10 pad 26: /sheet5F23178F/bus_3v3 -> (no net)
- J10 pad 3: /SPI1_SS -> /MOD4_SPI1_SS
- J10 pad 4: /SPI4_SS -> /MOD4_SPI2_SS
- J10 pad 6: /sheet5F23178F/UART2_RX -> /MOD4_UART2_RX
- J10 pad 7: Net-(J10-Pad7) -> (no net)
- J10 pad 8: /sheet5F23178F/bus_vbat -> (no net)
- J10 pad 9: /sheet5F23178F/bus_5v -> (no net)
- J12 pad 12: /SPI1_MOSI -> /MOD7_SPI1_MOSI
- J12 pad 13: /SPI4_MISO -> /MOD7_SPI2_MISO
- J12 pad 15: /sheet5F231790/UART1_TX -> /MOD7_UART1_TX
- J12 pad 16: Net-(J12-Pad16) -> (no net)
- J12 pad 17: Net-(J12-Pad17) -> (no net)
- J12 pad 2: /SPI1_MISO -> /MOD7_SPI1_MISO
- J12 pad 22: /SPI4_MOSI -> /MOD7_SPI2_MOSI
- J12 pad 23: /sheet5F231790/UART1_RX -> /MOD7_UART1_RX
- J12 pad 24: /sheet5F231790/UART2_TX -> /MOD7_UART2_TX
- J12 pad 25: Net-(J12-Pad25) -> (no net)
- J12 pad 26: /sheet5F231790/bus_3v3 -> (no net)
- J12 pad 3: /SPI1_SS -> /MOD7_SPI1_SS
- J12 pad 4: /SPI4_SS -> /MOD7_SPI2_SS
- J12 pad 6: /sheet5F231790/UART2_RX -> /MOD7_UART2_RX
- J12 pad 7: Net-(J12-Pad7) -> (no net)
- J12 pad 8: /sheet5F231790/bus_vbat -> (no net)
- J12 pad 9: /sheet5F231790/bus_5v -> (no net)
- J14 pad 12: /SPI1_MOSI -> /MOD8_SPI1_MOSI
- J14 pad 13: /SPI4_MISO -> /MOD8_SPI2_MISO
- J14 pad 15: /sheet5F237BCE/UART1_TX -> /MOD8_UART1_TX
- J14 pad 16: Net-(J14-Pad16) -> (no net)
- J14 pad 17: Net-(J14-Pad17) -> (no net)
- J14 pad 2: /SPI1_MISO -> /MOD8_SPI1_MISO
- J14 pad 22: /SPI4_MOSI -> /MOD8_SPI2_MOSI
- J14 pad 23: /sheet5F237BCE/UART1_RX -> /MOD8_UART1_RX
- J14 pad 24: /sheet5F237BCE/UART2_TX -> /MOD8_UART2_TX
- J14 pad 25: Net-(J14-Pad25) -> (no net)
- J14 pad 26: /sheet5F237BCE/bus_3v3 -> (no net)
- J14 pad 3: /SPI1_SS -> /MOD8_SPI1_SS
- J14 pad 4: /SPI4_SS -> /MOD8_SPI2_SS
- J14 pad 6: /sheet5F237BCE/UART2_RX -> /MOD8_UART2_RX
- J14 pad 7: Net-(J14-Pad7) -> (no net)
- J14 pad 8: /sheet5F237BCE/bus_vbat -> (no net)
- J14 pad 9: /sheet5F237BCE/bus_5v -> (no net)
- J16 pad 12: /SPI1_MOSI -> /MOD3_SPI1_MOSI
- J16 pad 13: /SPI4_MISO -> /MOD3_SPI2_MISO
- J16 pad 15: /sheet5F237BCF/UART1_TX -> /MOD3_UART1_TX
- J16 pad 16: Net-(J16-Pad16) -> (no net)
- J16 pad 17: Net-(J16-Pad17) -> (no net)
- J16 pad 2: /SPI1_MISO -> /MOD3_SPI1_MISO
- J16 pad 22: /SPI4_MOSI -> /MOD3_SPI2_MOSI
- J16 pad 23: /sheet5F237BCF/UART1_RX -> /MOD3_UART1_RX
- J16 pad 24: /sheet5F237BCF/UART2_TX -> /MOD3_UART2_TX
- J16 pad 25: Net-(J16-Pad25) -> (no net)
- J16 pad 26: /sheet5F237BCF/bus_3v3 -> (no net)
- J16 pad 3: /SPI1_SS -> /MOD3_SPI1_SS
- J16 pad 4: /SPI4_SS -> /MOD3_SPI2_SS
- J16 pad 6: /sheet5F237BCF/UART2_RX -> /MOD3_UART2_RX
- J16 pad 7: Net-(J16-Pad7) -> (no net)
- J16 pad 8: /sheet5F237BCF/bus_vbat -> (no net)
- J16 pad 9: /sheet5F237BCF/bus_5v -> (no net)
- J4 pad 12: /SPI1_MOSI -> /MOD5_SPI1_MOSI
- J4 pad 13: /SPI4_MISO -> /MOD5_SPI2_MISO
- J4 pad 15: /sheet5F22A1B0/UART1_TX -> /MOD5_UART1_TX
- J4 pad 16: Net-(J4-Pad16) -> (no net)
- J4 pad 17: Net-(J4-Pad17) -> (no net)
- J4 pad 2: /SPI1_MISO -> /MOD5_SPI1_MISO
- J4 pad 22: /SPI4_MOSI -> /MOD5_SPI2_MOSI
- J4 pad 23: /sheet5F22A1B0/UART1_RX -> /MOD5_UART1_RX
- J4 pad 24: /sheet5F22A1B0/UART2_TX -> /MOD5_UART2_TX
- J4 pad 25: Net-(J4-Pad25) -> (no net)
- J4 pad 26: /sheet5F22A1B0/bus_3v3 -> (no net)
- J4 pad 3: /SPI1_SS -> /MOD5_SPI1_SS
- J4 pad 4: /SPI4_SS -> /MOD5_SPI2_SS
- J4 pad 6: /sheet5F22A1B0/UART2_RX -> /MOD5_UART2_RX
- J4 pad 7: Net-(J4-Pad7) -> (no net)
- J4 pad 8: /sheet5F22A1B0/bus_vbat -> (no net)
- J4 pad 9: /sheet5F22A1B0/bus_5v -> (no net)
- J5 pad 1: /sheet5F22D1E9/UART1_RX -> /I2C2_SDA
- J5 pad 2: OBC_UART1_TX -> /MOD1_SPI1_MISO
- J5 pad 3: /sheet5F22D1E9/UART1_TX -> /MOD1_SPI1_SS
- J5 pad 4: OBC_UART1_RX -> /MOD1_SPI2_SS
- J5 pad 5: /sheet5F22D1E9/UART2_RX -> /CAN1_TX
- J5 pad 6: OBC_UART2_TX -> /MOD1_UART2_RX
- J5 pad 7: /sheet5F22D1E9/UART2_TX -> (no net)
- J5 pad 8: OBC_UART2_RX -> (no net)
- J6 pad 12: /SPI1_MOSI -> /MOD2_SPI1_MOSI
- J6 pad 13: /SPI4_MISO -> /MOD2_SPI2_MISO
- J6 pad 15: /sheet5F22D1E8/UART1_TX -> /MOD2_UART1_TX
- J6 pad 16: Net-(J6-Pad16) -> (no net)
- J6 pad 17: Net-(J6-Pad17) -> (no net)
- J6 pad 2: /SPI1_MISO -> /MOD2_SPI1_MISO
- J6 pad 22: /SPI4_MOSI -> /MOD2_SPI2_MOSI
- J6 pad 23: /sheet5F22D1E8/UART1_RX -> /MOD2_UART1_RX
- J6 pad 24: /sheet5F22D1E8/UART2_TX -> /MOD2_UART2_TX
- J6 pad 25: Net-(J6-Pad25) -> (no net)
- J6 pad 26: /sheet5F22D1E8/bus_3v3 -> (no net)
- J6 pad 3: /SPI1_SS -> /MOD2_SPI1_SS
- J6 pad 4: /SPI4_SS -> /MOD2_SPI2_SS
- J6 pad 6: /sheet5F22D1E8/UART2_RX -> /MOD2_UART2_RX
- J6 pad 7: Net-(J6-Pad7) -> (no net)
- J6 pad 8: /sheet5F22D1E8/bus_vbat -> (no net)
- J6 pad 9: /sheet5F22D1E8/bus_5v -> (no net)
- J8 pad 12: /SPI1_MOSI -> /MOD6_SPI1_MOSI
- J8 pad 13: /SPI4_MISO -> /MOD6_SPI2_MISO
- J8 pad 15: /sheet5F22D1E9/UART1_TX -> /MOD6_UART1_TX
- J8 pad 16: Net-(J8-Pad16) -> (no net)
- J8 pad 17: Net-(J8-Pad17) -> (no net)
- J8 pad 2: /SPI1_MISO -> /MOD6_SPI1_MISO
- J8 pad 22: /SPI4_MOSI -> /MOD6_SPI2_MOSI
- J8 pad 23: /sheet5F22D1E9/UART1_RX -> /MOD6_UART1_RX
- J8 pad 24: /sheet5F22D1E9/UART2_TX -> /MOD6_UART2_TX
- J8 pad 25: Net-(J8-Pad25) -> (no net)
- J8 pad 26: /sheet5F22D1E9/bus_3v3 -> (no net)
- J8 pad 3: /SPI1_SS -> /MOD6_SPI1_SS
- J8 pad 4: /SPI4_SS -> /MOD6_SPI2_SS
- J8 pad 6: /sheet5F22D1E9/UART2_RX -> /MOD6_UART2_RX
- J8 pad 7: Net-(J8-Pad7) -> (no net)
- J8 pad 8: /sheet5F22D1E9/bus_vbat -> (no net)
- J8 pad 9: /sheet5F22D1E9/bus_5v -> (no net)
- R1 pad 1: GND -> /Sheet5F4EF57F/VBAT
- R1 pad 2: Net-(D1-Pad1) -> /Sheet5F4EF57F/Sheet5F4EF936/EN
- R2 pad 1: GND -> /Sheet5F4EF57F/Sheet5F4EF936/EN
- R2 pad 2: Net-(D2-Pad1) -> GND
- R3 pad 1: GND -> Net-(R3-Pad1)
- R3 pad 2: Net-(D3-Pad1) -> GND
- SW10 pad 1: /Vin -> GND
- SW10 pad 2: Vbat -> GND
Routing:
- net /SPI1_SCK: track 0.00 -> 511.4 mm
- net /I2C2_SDA: track 0.00 -> 505.6 mm
- net /SPI4_SCK: track 0.00 -> 504.1 mm
- net /I2C1_SCL: track 0.00 -> 501.5 mm
- net /I2C1_SDA: track 0.00 -> 500.2 mm
- net /I2C2_SCL: track 0.00 -> 491.3 mm
- net /CAN1_RX: track 0.00 -> 467.8 mm
- net /CAN1_TX: track 0.00 -> 449.0 mm
- net /MOD6_UART2_TX: track 0.00 -> 75.8 mm
- net /MOD7_UART2_TX: track 0.00 -> 74.7 mm
- net /MOD3_UART2_TX: track 0.00 -> 74.5 mm
- net /MOD2_UART2_TX: track 0.00 -> 74.2 mm
- net /MOD1_UART2_TX: track 0.00 -> 73.2 mm
- net /MOD5_UART2_TX: track 0.00 -> 73.0 mm
- net /MOD8_UART2_TX: track 0.00 -> 72.8 mm
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- added copper zone on B.Cu, net /Sheet5F4EF57F/3.3V
- added copper zone on B.Cu, net /Sheet5F4EF57F/5V
- added copper zone on B.Cu, net /Sheet5F4EF57F/Sheet5F698D24/5V
- added copper zone on F.Cu, net Net-(C15-Pad1)
- added copper zone on F.Cu, net Net-(C5-Pad1)
- added copper zone on F.Cu, net Net-(C52-Pad1)
Other:
- rule via_min_drill: 0.3 -> 0.25
- rule via_min_size: 0.4 -> 0.6
- board text added: "[7V-60V]"
- board text removed: "[9V-14V]"

Commit message: Most PSB done, needs more silk screen cosmetic plus review
Signed-off-by: Alexis Jeandet <alexis.jeandet@member.fsf.org>
Parts:
- added C58: C, Capacitor_SMD:C_0603_1608Metric_Pad1.05x0.95mm_HandSolder, B.Cu at (28.7, 88.1)
- added C59: C, Capacitor_SMD:C_0603_1608Metric_Pad1.05x0.95mm_HandSolder, F.Cu at (29.2, 93.3)
- added C60: C, Capacitor_SMD:C_0603_1608Metric_Pad1.05x0.95mm_HandSolder, B.Cu at (151.3, 63.4)
- added C61: C, Capacitor_SMD:C_0603_1608Metric_Pad1.05x0.95mm_HandSolder, F.Cu at (147.6, 60.9)
- added C62: C, Capacitor_SMD:C_0603_1608Metric_Pad1.05x0.95mm_HandSolder, B.Cu at (38.0, 138.4)
- added C63: C, Capacitor_SMD:C_0603_1608Metric_Pad1.05x0.95mm_HandSolder, F.Cu at (41.9, 142.4)
- added C64: C, Capacitor_SMD:C_0603_1608Metric_Pad1.05x0.95mm_HandSolder, B.Cu at (57.3, 46.7)
- added C65: C, Capacitor_SMD:C_0603_1608Metric_Pad1.05x0.95mm_HandSolder, F.Cu at (54.9, 48.4)
- added C66: C, Capacitor_SMD:C_0603_1608Metric_Pad1.05x0.95mm_HandSolder, B.Cu at (81.8, 167.5)
- added C67: C, Capacitor_SMD:C_0603_1608Metric_Pad1.05x0.95mm_HandSolder, F.Cu at (86.7, 167.1)
- added C68: C, Capacitor_SMD:C_0603_1608Metric_Pad1.05x0.95mm_HandSolder, B.Cu at (133.6, 157.5)
- added C69: C, Capacitor_SMD:C_0603_1608Metric_Pad1.05x0.95mm_HandSolder, F.Cu at (135.8, 153.3)
- added C70: C, Capacitor_SMD:C_0603_1608Metric_Pad1.05x0.95mm_HandSolder, B.Cu at (107.4, 36.1)
- added C71: C, Capacitor_SMD:C_0603_1608Metric_Pad1.05x0.95mm_HandSolder, F.Cu at (103.6, 35.3)
- added C72: C, Capacitor_SMD:C_0603_1608Metric_Pad1.05x0.95mm_HandSolder, B.Cu at (162.0, 115.1)
- added C73: C, Capacitor_SMD:C_0603_1608Metric_Pad1.05x0.95mm_HandSolder, F.Cu at (161.9, 111.1)
- added J2: Conn_01x06, Connector_PinHeader_2.54mm:PinHeader_1x06_P2.54mm_Vertical, F.Cu at (121.0, 90.8)
- added J3: Conn_01x06, Connector_PinHeader_2.54mm:PinHeader_1x06_P2.54mm_Vertical, F.Cu at (93.2, 74.1)
- added R28: R, Resistor_SMD:R_0603_1608Metric_Pad1.05x0.95mm_HandSolder, F.Cu at (42.4, 95.6)
- added R29: R, Resistor_SMD:R_0603_1608Metric_Pad1.05x0.95mm_HandSolder, F.Cu at (42.4, 93.0)
- added R30: R, Resistor_SMD:R_1210_3225Metric_Pad1.42x2.65mm_HandSolder, B.Cu at (25.4, 91.4)
- added R31: R, Resistor_SMD:R_1210_3225Metric_Pad1.42x2.65mm_HandSolder, F.Cu at (25.9, 89.8)
- added R32: R, Resistor_SMD:R_0603_1608Metric_Pad1.05x0.95mm_HandSolder, F.Cu at (42.4, 98.1)
- added R33: R, Resistor_SMD:R_0603_1608Metric_Pad1.05x0.95mm_HandSolder, B.Cu at (33.8, 96.3)
- added R34: R, Resistor_SMD:R_0603_1608Metric_Pad1.05x0.95mm_HandSolder, F.Cu at (136.2, 68.5)
- added R35: R, Resistor_SMD:R_0603_1608Metric_Pad1.05x0.95mm_HandSolder, F.Cu at (137.9, 70.3)
- added R36: R, Resistor_SMD:R_1210_3225Metric_Pad1.42x2.65mm_HandSolder, B.Cu at (151.3, 58.7)
- added R37: R, Resistor_SMD:R_1210_3225Metric_Pad1.42x2.65mm_HandSolder, F.Cu at (152.2, 60.9)
- added R38: R, Resistor_SMD:R_0603_1608Metric_Pad1.05x0.95mm_HandSolder, F.Cu at (134.3, 66.7)
- added R39: R, Resistor_SMD:R_0603_1608Metric_Pad1.05x0.95mm_HandSolder, B.Cu at (144.3, 60.0)
- added R40: R, Resistor_SMD:R_0603_1608Metric_Pad1.05x0.95mm_HandSolder, F.Cu at (53.4, 134.8)
- added R41: R, Resistor_SMD:R_0603_1608Metric_Pad1.05x0.95mm_HandSolder, F.Cu at (51.6, 133.0)
- added R42: R, Resistor_SMD:R_1210_3225Metric_Pad1.42x2.65mm_HandSolder, B.Cu at (38.0, 143.1)
- added R43: R, Resistor_SMD:R_1210_3225Metric_Pad1.42x2.65mm_HandSolder, F.Cu at (37.2, 142.3)
- added R44: R, Resistor_SMD:R_0603_1608Metric_Pad1.05x0.95mm_HandSolder, F.Cu at (55.3, 136.7)
- added R45: R, Resistor_SMD:R_0603_1608Metric_Pad1.05x0.95mm_HandSolder, B.Cu at (48.9, 141.7)
- added R46: R, Resistor_SMD:R_0603_1608Metric_Pad1.05x0.95mm_HandSolder, F.Cu at (62.1, 59.7)
- added R47: R, Resistor_SMD:R_0603_1608Metric_Pad1.05x0.95mm_HandSolder, F.Cu at (63.8, 58.0)
- added R48: R, Resistor_SMD:R_1210_3225Metric_Pad1.42x2.65mm_HandSolder, B.Cu at (52.7, 46.7)
- added R49: R, Resistor_SMD:R_1210_3225Metric_Pad1.42x2.65mm_HandSolder, F.Cu at (54.9, 43.8)
- added R50: R, Resistor_SMD:R_0603_1608Metric_Pad1.05x0.95mm_HandSolder, F.Cu at (60.3, 61.5)
- added R51: R, Resistor_SMD:R_0603_1608Metric_Pad1.05x0.95mm_HandSolder, B.Cu at (52.9, 53.8)
- added R52: R, Resistor_SMD:R_0603_1608Metric_Pad1.05x0.95mm_HandSolder, F.Cu at (89.2, 154.2)
- added R53: R, Resistor_SMD:R_0603_1608Metric_Pad1.05x0.95mm_HandSolder, F.Cu at (86.6, 154.2)
- added R54: R, Resistor_SMD:R_1210_3225Metric_Pad1.42x2.65mm_HandSolder, B.Cu at (85.1, 170.7)
- added R55: R, Resistor_SMD:R_1210_3225Metric_Pad1.42x2.65mm_HandSolder, F.Cu at (83.4, 170.4)
- added R56: R, Resistor_SMD:R_0603_1608Metric_Pad1.05x0.95mm_HandSolder, F.Cu at (91.7, 154.2)
- added R57: R, Resistor_SMD:R_0603_1608Metric_Pad1.05x0.95mm_HandSolder, B.Cu at (90.8, 162.5)
- added R58: R, Resistor_SMD:R_0603_1608Metric_Pad1.05x0.95mm_HandSolder, F.Cu at (128.0, 143.0)
- added R59: R, Resistor_SMD:R_0603_1608Metric_Pad1.05x0.95mm_HandSolder, F.Cu at (126.2, 144.8)
- added R60: R, Resistor_SMD:R_1210_3225Metric_Pad1.42x2.65mm_HandSolder, B.Cu at (138.3, 157.5)
- added R61: R, Resistor_SMD:R_1210_3225Metric_Pad1.42x2.65mm_HandSolder, F.Cu at (135.7, 158.0)
- added R62: R, Resistor_SMD:R_0603_1608Metric_Pad1.05x0.95mm_HandSolder, F.Cu at (129.8, 141.2)
- added R63: R, Resistor_SMD:R_0603_1608Metric_Pad1.05x0.95mm_HandSolder, B.Cu at (137.4, 150.0)
- added R64: R, Resistor_SMD:R_0603_1608Metric_Pad1.05x0.95mm_HandSolder, F.Cu at (100.9, 49.1)
- added R65: R, Resistor_SMD:R_0603_1608Metric_Pad1.05x0.95mm_HandSolder, F.Cu at (103.4, 49.1)
- added R66: R, Resistor_SMD:R_1210_3225Metric_Pad1.42x2.65mm_HandSolder, B.Cu at (104.1, 32.8)
- added R67: R, Resistor_SMD:R_1210_3225Metric_Pad1.42x2.65mm_HandSolder, F.Cu at (106.9, 32.1)
- added R68: R, Resistor_SMD:R_0603_1608Metric_Pad1.05x0.95mm_HandSolder, F.Cu at (98.3, 49.1)
- added R69: R, Resistor_SMD:R_0603_1608Metric_Pad1.05x0.95mm_HandSolder, B.Cu at (99.6, 37.5)
- added R70: R, Resistor_SMD:R_0603_1608Metric_Pad1.05x0.95mm_HandSolder, F.Cu at (159.1, 107.2)
- added R71: R, Resistor_SMD:R_0603_1608Metric_Pad1.05x0.95mm_HandSolder, F.Cu at (159.1, 109.8)
- added R72: R, Resistor_SMD:R_1210_3225Metric_Pad1.42x2.65mm_HandSolder, B.Cu at (165.3, 111.8)
- added R73: R, Resistor_SMD:R_1210_3225Metric_Pad1.42x2.65mm_HandSolder, F.Cu at (165.2, 114.4)
- added R74: R, Resistor_SMD:R_0603_1608Metric_Pad1.05x0.95mm_HandSolder, F.Cu at (159.1, 104.7)
- added R75: R, Resistor_SMD:R_0603_1608Metric_Pad1.05x0.95mm_HandSolder, B.Cu at (160.5, 107.7)
- added SW1: SW_DIP_x03, Button_Switch_THT:SW_DIP_SPSTx03_Slide_9.78x9.8mm_W7.62mm_P2.54mm, F.Cu at (53.6, 98.1)
- added SW2: SW_DIP_x03, Button_Switch_THT:SW_DIP_SPSTx03_Slide_9.78x9.8mm_W7.62mm_P2.54mm, F.Cu at (126.3, 74.7)
- added SW3: SW_DIP_x03, Button_Switch_THT:SW_DIP_SPSTx03_Slide_9.78x9.8mm_W7.62mm_P2.54mm, F.Cu at (63.3, 128.6)
- added SW4: SW_DIP_x03, Button_Switch_THT:SW_DIP_SPSTx03_Slide_9.78x9.8mm_W7.62mm_P2.54mm, F.Cu at (68.3, 69.6)
- added SW5: SW_DIP_x03, Button_Switch_THT:SW_DIP_SPSTx03_Slide_9.78x9.8mm_W7.62mm_P2.54mm, F.Cu at (91.7, 142.8)
- added SW6: SW_DIP_x03, Button_Switch_THT:SW_DIP_SPSTx03_Slide_9.78x9.8mm_W7.62mm_P2.54mm, F.Cu at (121.7, 133.1)
- added SW7: SW_DIP_x03, Button_Switch_THT:SW_DIP_SPSTx03_Slide_9.78x9.8mm_W7.62mm_P2.54mm, F.Cu at (98.3, 60.5)
- added SW8: SW_DIP_x03, Button_Switch_THT:SW_DIP_SPSTx03_Slide_9.78x9.8mm_W7.62mm_P2.54mm, F.Cu at (147.6, 104.7)
- added U10: TPS22917DBV, Package_TO_SOT_SMD:SOT-23-6, F.Cu at (26.6, 93.4)
- added U11: BTS6163D, Package_TO_SOT_SMD:TO-252-4, B.Cu at (29.5, 100.5)
- added U12: TPS22917DBV, Package_TO_SOT_SMD:SOT-23-6, B.Cu at (153.3, 61.7)
- added U13: TPS22917DBV, Package_TO_SOT_SMD:SOT-23-6, F.Cu at (149.2, 58.8)
- added U14: BTS6163D, Package_TO_SOT_SMD:TO-252-4, B.Cu at (144.1, 53.6)
- added U15: TPS22917DBV, Package_TO_SOT_SMD:SOT-23-6, B.Cu at (36.0, 140.1)
- added U16: TPS22917DBV, Package_TO_SOT_SMD:SOT-23-6, F.Cu at (40.2, 144.4)
- added U17: BTS6163D, Package_TO_SOT_SMD:TO-252-4, B.Cu at (48.9, 147.8)
- added U18: TPS22917DBV, Package_TO_SOT_SMD:SOT-23-6, B.Cu at (55.6, 44.6)
- added U19: TPS22917DBV, Package_TO_SOT_SMD:SOT-23-6, F.Cu at (52.9, 46.8)
- added U20: BTS6163D, Package_TO_SOT_SMD:TO-252-4, B.Cu at (46.6, 53.9)
- added U21: TPS22917DBV, Package_TO_SOT_SMD:SOT-23-6, B.Cu at (81.5, 170.1)
- added U22: TPS22917DBV, Package_TO_SOT_SMD:SOT-23-6, F.Cu at (86.9, 169.7)
- added U23: BTS6163D, Package_TO_SOT_SMD:TO-252-4, B.Cu at (95.4, 166.9)
- added U24: TPS22917DBV, Package_TO_SOT_SMD:SOT-23-6, B.Cu at (135.3, 159.6)
- added U25: TPS22917DBV, Package_TO_SOT_SMD:SOT-23-6, F.Cu at (137.8, 155.0)
- added U26: BTS6163D, Package_TO_SOT_SMD:TO-252-4, B.Cu at (143.5, 150.0)
- added U27: TPS22917DBV, Package_TO_SOT_SMD:SOT-23-6, B.Cu at (107.6, 33.5)
- added U28: TPS22917DBV, Package_TO_SOT_SMD:SOT-23-6, F.Cu at (103.4, 32.7)
- added U29: BTS6163D, Package_TO_SOT_SMD:TO-252-4, B.Cu at (94.9, 33.1)
- added U30: TPS22917DBV, Package_TO_SOT_SMD:SOT-23-6, B.Cu at (164.6, 115.4)
- added U31: TPS22917DBV, Package_TO_SOT_SMD:SOT-23-6, F.Cu at (164.5, 110.9)
- added U32: BTS6163D, Package_TO_SOT_SMD:TO-252-4, B.Cu at (164.9, 103.1)
- added U9: TPS22917DBV, Package_TO_SOT_SMD:SOT-23-6, B.Cu at (26.0, 87.8)
- moved L4 0.28 mm to (115.3, 108.7)
Connections:
- net /Sheet5F4EF57F/3.3V renamed /3.3V
- net /Sheet5F4EF57F/5V renamed /5V
- net /Sheet5F4EF57F/VBAT renamed /VBAT
- J10 pad 17: (no net) -> /sheet5F23178F/bus_vbat
- J10 pad 26: (no net) -> /sheet5F23178F/bus_3v3
- J10 pad 8: (no net) -> /sheet5F23178F/bus_vbat
- J10 pad 9: (no net) -> /sheet5F23178F/bus_5v
- J12 pad 17: (no net) -> /sheet5F231790/bus_vbat
- J12 pad 26: (no net) -> /sheet5F231790/bus_3v3
- J12 pad 8: (no net) -> /sheet5F231790/bus_vbat
- J12 pad 9: (no net) -> /sheet5F231790/bus_5v
- J14 pad 17: (no net) -> /sheet5F237BCE/bus_vbat
- J14 pad 26: (no net) -> /sheet5F237BCE/bus_3v3
- J14 pad 8: (no net) -> /sheet5F237BCE/bus_vbat
- J14 pad 9: (no net) -> /sheet5F237BCE/bus_5v
- J16 pad 17: (no net) -> /sheet5F237BCF/bus_vbat
- J16 pad 26: (no net) -> /sheet5F237BCF/bus_3v3
- J16 pad 8: (no net) -> /sheet5F237BCF/bus_vbat
- J16 pad 9: (no net) -> /sheet5F237BCF/bus_5v
- J4 pad 17: (no net) -> /sheet5F22A1B0/bus_vbat
- J4 pad 26: (no net) -> /sheet5F22A1B0/bus_3v3
- J4 pad 8: (no net) -> /sheet5F22A1B0/bus_vbat
- J4 pad 9: (no net) -> /sheet5F22A1B0/bus_5v
- J5 pad 17: (no net) -> /sheet5F66A269/bus_vbat
- J5 pad 26: (no net) -> /sheet5F66A269/bus_3v3
- J5 pad 8: (no net) -> /sheet5F66A269/bus_vbat
- J5 pad 9: (no net) -> /sheet5F66A269/bus_5v
- J6 pad 17: (no net) -> /sheet5F22D1E8/bus_vbat
- J6 pad 26: (no net) -> /sheet5F22D1E8/bus_3v3
- J6 pad 8: (no net) -> /sheet5F22D1E8/bus_vbat
- J6 pad 9: (no net) -> /sheet5F22D1E8/bus_5v
- J8 pad 17: (no net) -> /sheet5F22D1E9/bus_vbat
- J8 pad 26: (no net) -> /sheet5F22D1E9/bus_3v3
- J8 pad 8: (no net) -> /sheet5F22D1E9/bus_vbat
- J8 pad 9: (no net) -> /sheet5F22D1E9/bus_5v
- U4 pad 102: (no net) -> /Sheet5F604EE5/IO8
- U4 pad 104: /MOD2_UART2_TX -> /Sheet5F604EE5/IO1
- U4 pad 105: /MOD2_UART1_TX -> /Sheet5F604EE5/IO2
- U4 pad 106: /MOD2_UART2_RX -> /Sheet5F604EE5/IO3
- U4 pad 107: /MOD2_UART1_RX -> /Sheet5F604EE5/IO4
- U4 pad 112: /MOD2_SPI2_MOSI -> /MOD2_UART2_TX
- U4 pad 113: /MOD2_SPI2_SS -> /MOD2_UART1_TX
- U4 pad 114: /MOD2_SPI2_MISO -> /MOD2_UART2_RX
- U4 pad 115: /MOD2_SPI1_SS -> /MOD2_UART1_RX
- U4 pad 116: /MOD2_SPI1_MOSI -> /MOD2_SPI2_MOSI
- U4 pad 117: /MOD2_SPI1_MISO -> /MOD2_SPI2_SS
- U4 pad 118: (no net) -> /MOD2_SPI2_MISO
- U4 pad 119: (no net) -> /MOD2_SPI1_SS
- U4 pad 120: (no net) -> /MOD2_SPI1_MOSI
- U4 pad 121: (no net) -> /MOD2_SPI1_MISO
- U4 pad 122: (no net) -> /Sheet5F604EE5/IO7
- U4 pad 128: (no net) -> /Sheet5F604EE5/IO6
- U4 pad 129: (no net) -> /Sheet5F604EE5/IO5
Routing:
- net /3.3V: track 0.90 -> 541.4 mm, vias 1 -> 4
- net /5V: track 0.90 -> 527.0 mm
- net /MOD8_SPI1_MOSI: track 0.00 -> 69.6 mm
- net /Sheet5F4EF57F/Sheet5F698D24/5V: track 12.3 -> 50.8 mm, vias 3 -> 5
- net VCCIO_0: track 26.4 -> 64.3 mm, vias 11 -> 16
- net /sheet5F22D1E8/5V_SW: track 0.00 -> 26.6 mm
- net /sheet5F237BCE/5V_SW: track 0.00 -> 26.3 mm
- net /sheet5F22D1E9/5V_SW: track 0.00 -> 26.1 mm
- net /sheet5F231790/5V_SW: track 0.00 -> 25.7 mm
- net /Sheet5F604EE5/IO8: track 0.00 -> 25.6 mm, vias 0 -> 1
- net /sheet5F22A1B0/5V_SW: track 0.00 -> 25.5 mm
- net /sheet5F237BCF/5V_SW: track 0.00 -> 25.1 mm
- net /sheet5F23178F/5V_SW: track 0.00 -> 24.4 mm
- net /sheet5F22A1B0/3.3V_SW: track 0.00 -> 21.5 mm
- net /sheet5F237BCF/3.3V_SW: track 0.00 -> 21.2 mm
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- added copper zone on B.Cu, net /VBAT
- added copper zone on In1.Cu, net /VBAT
- added copper zone on In2.Cu, net /VBAT
- added copper zone on B.Cu, net GND
- added copper zone on In1.Cu, net GND
- added copper zone on In2.Cu, net GND
- added copper zone on In1.Cu, net VCC
- added copper zone on In2.Cu, net VCCIO_0
- removed copper zone on In2.Cu, net 3V3
- removed copper zone on B.Cu, net 5V
- removed copper zone on In1.Cu, net Vbat
Other:
- board text removed: "OBC"
- board text removed: "UART1_RX"
- board text removed: "UART1_TX"
- board text removed: "UART2_RX"
- board text removed: "UART2_TX"

Commit message: added some text, moved headers, added X logo, fixed res/diode overlap, fixed DRC
Parts:
- added LOGO1: LOGO, FlatSatHub:X-LOGO, F.Cu at (35.7, 120.4)
- moved J17 12.5 mm to (116.0, 122.9), turned to 315 degrees
- moved J2 11.5 mm to (116.0, 80.4), turned to 45 degrees
- moved J3 2.88 mm to (94.8, 71.7)
- moved C43 1.08 mm to (119.1, 106.1)
Connections:
- J10 pad 16: (no net) -> Net-(J10-Pad16)
- J10 pad 25: (no net) -> Net-(J10-Pad25)
- J10 pad 7: (no net) -> Net-(J10-Pad7)
- J12 pad 16: (no net) -> Net-(J12-Pad16)
- J12 pad 25: (no net) -> Net-(J12-Pad25)
- J12 pad 7: (no net) -> Net-(J12-Pad7)
- J14 pad 16: (no net) -> Net-(J14-Pad16)
- J14 pad 25: (no net) -> Net-(J14-Pad25)
- J14 pad 7: (no net) -> Net-(J14-Pad7)
- J16 pad 16: (no net) -> Net-(J16-Pad16)
- J16 pad 25: (no net) -> Net-(J16-Pad25)
- J16 pad 7: (no net) -> Net-(J16-Pad7)
- J4 pad 16: (no net) -> Net-(J4-Pad16)
- J4 pad 25: (no net) -> Net-(J4-Pad25)
- J4 pad 7: (no net) -> Net-(J4-Pad7)
- J5 pad 16: (no net) -> Net-(J5-Pad16)
- J5 pad 25: (no net) -> Net-(J5-Pad25)
- J5 pad 7: (no net) -> Net-(J5-Pad7)
- J6 pad 16: (no net) -> Net-(J6-Pad16)
- J6 pad 25: (no net) -> Net-(J6-Pad25)
- J6 pad 7: (no net) -> Net-(J6-Pad7)
- J8 pad 16: (no net) -> Net-(J8-Pad16)
- J8 pad 25: (no net) -> Net-(J8-Pad25)
- J8 pad 7: (no net) -> Net-(J8-Pad7)
- U3 pad 1: (no net) -> Net-(U3-Pad1)
- U4 pad 109: (no net) -> Net-(U4-Pad109)
- U4 pad 110: (no net) -> Net-(U4-Pad110)
- U4 pad 124: (no net) -> Net-(U4-Pad124)
- U4 pad 125: (no net) -> Net-(U4-Pad125)
- U4 pad 130: (no net) -> Net-(U4-Pad130)
- U4 pad 15: (no net) -> Net-(U4-Pad15)
- U4 pad 16: (no net) -> Net-(U4-Pad16)
- U4 pad 17: (no net) -> Net-(U4-Pad17)
- U4 pad 18: (no net) -> Net-(U4-Pad18)
- U4 pad 55: (no net) -> Net-(U4-Pad55)
- U4 pad 77: (no net) -> Net-(U4-Pad77)
- U4 pad 82: (no net) -> Net-(U4-Pad82)
- U4 pad 83: (no net) -> Net-(U4-Pad83)
- U4 pad 84: (no net) -> Net-(U4-Pad84)
- U4 pad 85: (no net) -> Net-(U4-Pad85)
- U7 pad 4: (no net) -> Net-(U7-Pad4)
Routing:
- net GND: track 5.19 -> 33.6 mm, vias 44 -> 45
- net /Sheet5F604EE5/FLASH_~CRESET: track 23.7 -> 37.2 mm, vias 1 -> 2
- net /Sheet5F604EE5/FLASH_CLK: track 27.2 -> 36.2 mm
- net /Sheet5F604EE5/FLASH_MOSI: track 26.4 -> 35.0 mm
- net /Sheet5F604EE5/FLASH_CS: track 29.4 -> 37.8 mm
- net /Sheet5F604EE5/FLASH_MISO: track 23.8 -> 31.3 mm
- net /Sheet5F604EE5/IO4: track 13.6 -> 19.9 mm, vias 0 -> 1
- net /Sheet5F604EE5/IO3: track 14.8 -> 19.3 mm, vias 0 -> 1
- net /Sheet5F604EE5/IO1: track 17.3 -> 20.8 mm
- net /Sheet5F604EE5/IO6: track 17.7 -> 20.9 mm
- net /Sheet5F604EE5/IO7: track 17.5 -> 20.7 mm
- net /Sheet5F604EE5/IO8: track 25.6 -> 28.7 mm
- net /Sheet5F604EE5/IO5: track 17.0 -> 19.9 mm
- net VCCIO_0: track 64.3 -> 61.9 mm
- net /Sheet5F604EE5/IO2: track 16.1 -> 18.1 mm, vias 0 -> 1
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Other:
- board text added: "3.3V"
- board text added: "MASTER"
