File: TPS54560.sch (KiCad schematic (older format))
At the start: 19 parts, among them U1 TPS54560B

Commit message: Most PSB done, needs more silk screen cosmetic plus review
Signed-off-by: Alexis Jeandet <alexis.jeandet@member.fsf.org>
Changed lines of the file:
@@
 $Descr A4 11693 8268
 encoding utf-8
-Sheet 10 15
+Sheet 13 15
 Title ""
 Date ""
@@
 AR Path="/5F4EF580/5F54C416/5F4F0601" Ref="U2"  Part="1"
 AR Path="/5F4EF580/5F69D9D1/5F4F0601" Ref="U8"  Part="1"
-F 0 "U1" H 5425 5740 50  0000 C CNN
+F 0 "U8" H 5425 5740 50  0000 C CNN
 F 1 "TPS54560B" H 5425 5649 50  0000 C CNB
 F 2 "Package_SO:Texas_R-PDSO-G8_EP2.95x4.9mm_Mask2.4x3.1mm" H 4875 4325 50  0001 C CNN
@@
 AR Path="/5F4EF580/5F54C416/5F4F0C59" Ref="C15"  Part="1"
 AR Path="/5F4EF580/5F69D9D1/5F4F0C59" Ref="C52"  Part="1"
-F 0 "C5" V 5098 2575 50  0000 C CNN
+F 0 "C52" V 5098 2575 50  0000 C CNN
 F 1 "C" V 5189 2575 50  0000 C CNN
 F 2 "Capacitor_SMD:C_0603_1608Metric_Pad1.05x0.95mm_HandSolder" H 5388 2425 50  0001 C CNN
@@
 AR Path="/5F4EF580/5F54C416/5F4F1384" Ref="C18"  Part="1"
 AR Path="/5F4EF580/5F69D9D1/5F4F1384" Ref="C55"  Part="1"
-F 0 "C8" H 7440 3421 50  0000 L CNN
+F 0 "C55" H 7440 3421 50  0000 L CNN
 F 1 "47u" H 7440 3330 50  0000 L CNN
 F 2 "Capacitor_SMD:C_1210_3225Metric_Pad1.42x2.65mm_HandSolder" H 7363 3225 50  0001 C CNN
@@
 AR Path="/5F4EF580/5F54C416/5F4F23F8" Ref="C19"  Part="1"
 AR Path="/5F4EF580/5F69D9D1/5F4F23F8" Ref="C56"  Part="1"
-F 0 "C9" H 7865 3421 50  0000 L CNN
+F 0 "C56" H 7865 3421 50  0000 L CNN
 F 1 "47u" H 7865 3330 50  0000 L CNN
 F 2 "Capacitor_SMD:C_1210_3225Metric_Pad1.42x2.65mm_HandSolder" H 7788 3225 50  0001 C CNN
@@
 AR Path="/5F4EF580/5F54C416/5F4F2834" Ref="C20"  Part="1"
 AR Path="/5F4EF580/5F69D9D1/5F4F2834" Ref="C57"  Part="1"
-F 0 "C10" H 8315 3421 50  0000 L CNN
+F 0 "C57" H 8315 3421 50  0000 L CNN
 F 1 "47u" H 8315 3330 50  0000 L CNN
 F 2 "Capacitor_SMD:C_1210_3225Metric_Pad1.42x2.65mm_HandSolder" H 8238 3225 50  0001 C CNN
@@
 AR Path="/5F4EF580/5F54C416/5F4F2E60" Ref="L2"  Part="1"
 AR Path="/5F4EF580/5F69D9D1/5F4F2E60" Ref="L5"  Part="1"
-F 0 "L1" V 6790 3175 50  0000 C CNN
+F 0 "L5" V 6790 3175 50  0000 C CNN
 F 1 "7.2uH" V 6699 3175 50  0000 C CNN
 F 2 "Inductor_SMD:L_Wuerth_HCI-1040" H 6600 3175 50  0001 C CNN
@@
 AR Path="/5F4EF580/5F54C416/5F5180E1" Ref="D2"  Part="1"
 AR Path="/5F4EF580/5F69D9D1/5F5180E1" Ref="D5"  Part="1"
-F 0 "D1" V 6275 3455 50  0000 L CNN
+F 0 "D5" V 6275 3455 50  0000 L CNN
 F 1 "D_Schottky" V 6320 3455 50  0001 L CNN
 F 2 "Diode_SMD:D_SMC_Handsoldering" H 6275 3375 50  0001 C CNN
@@
 AR Path="/5F4EF580/5F54C416/5F519486" Ref="R11"  Part="1"
 AR Path="/5F4EF580/5F69D9D1/5F519486" Ref="R26"  Part="1"
-F 0 "R5" H 7045 3421 50  0000 L CNN
+F 0 "R26" H 7045 3421 50  0000 L CNN
 F 1 "R" H 7045 3330 50  0000 L CNN
 F 2 "Resistor_SMD:R_0603_1608Metric_Pad1.05x0.95mm_HandSolder" V 6905 3375 50  0001 C CNN
@@
 AR Path="/5F4EF580/5F54C416/5F519CE5" Ref="R12"  Part="1"
 AR Path="/5F4EF580/5F69D9D1/5F519CE5" Ref="R27"  Part="1"
-F 0 "R6" H 7045 3946 50  0000 L CNN
+F 0 "R27" H 7045 3946 50  0000 L CNN
 F 1 "R" H 7045 3855 50  0000 L CNN
 F 2 "Resistor_SMD:R_0603_1608Metric_Pad1.05x0.95mm_HandSolder" V 6905 3900 50  0001 C CNN
@@
 AR Path="/5F4EF580/5F54C416/5F521EA6" Ref="R10"  Part="1"
 AR Path="/5F4EF580/5F69D9D1/5F521EA6" Ref="R25"  Part="1"
-F 0 "R4" H 6445 4471 50  0000 L CNN
+F 0 "R25" H 6445 4471 50  0000 L CNN
 F 1 "R" H 6445 4380 50  0000 L CNN
 F 2 "Resistor_SMD:R_0603_1608Metric_Pad1.05x0.95mm_HandSolder" V 6305 4425 50  0001 C CNN
@@
 AR Path="/5F4EF580/5F54C416/5F52270E" Ref="C17"  Part="1"
 AR Path="/5F4EF580/5F69D9D1/5F52270E" Ref="C54"  Part="1"
-F 0 "C7" V 6523 4600 50  0000 C CNN
+F 0 "C54" V 6523 4600 50  0000 C CNN
 F 1 "C" V 6614 4600 50  0000 C CNN
 F 2 "Capacitor_SMD:C_0603_1608Metric_Pad1.05x0.95mm_HandSolder" H 6813 4450 50  0001 C CNN
@@
 AR Path="/5F4EF580/5F54C416/5F524117" Ref="C16"  Part="1"
 AR Path="/5F4EF580/5F69D9D1/5F524117" Ref="C53"  Part="1"
-F 0 "C6" V 6123 4850 50  0000 C CNN
+F 0 "C53" V 6123 4850 50  0000 C CNN
 F 1 "C" V 6214 4850 50  0000 C CNN
 F 2 "Capacitor_SMD:C_0603_1608Metric_Pad1.05x0.95mm_HandSolder" H 6413 4700 50  0001 C CNN
@@
 AR Path="/5F4EF580/5F54C416/5F5286A3" Ref="R9"  Part="1"
 AR Path="/5F4EF580/5F69D9D1/5F5286A3" Ref="R24"  Part="1"
-F 0 "R3" H 4745 4521 50  0000 L CNN
+F 0 "R24" H 4745 4521 50  0000 L CNN
 F 1 "R" H 4745 4430 50  0000 L CNN
 F 2 "Resistor_SMD:R_0603_1608Metric_Pad1.05x0.95mm_HandSolder" V 4605 4475 50  0001 C CNN
@@
 AR Path="/5F4EF580/5F54C416/5F52B4B6" Ref="C14"  Part="1"
 AR Path="/5F4EF580/5F69D9D1/5F52B4B6" Ref="C51"  Part="1"
-F 0 "C4" H 3915 3646 50  0000 L CNN
+F 0 "C51" H 3915 3646 50  0000 L CNN
 F 1 "2.2uF" H 3915 3555 50  0000 L CNN
 F 2 "Capacitor_SMD:C_1210_3225Metric_Pad1.42x2.65mm_HandSolder" H 3838 3450 50  0001 C CNN
@@
 AR Path="/5F4EF580/5F54C416/5F52C663" Ref="C13"  Part="1"
 AR Path="/5F4EF580/5F69D9D1/5F52C663" Ref="C50"  Part="1"
-F 0 "C3" H 3465 3646 50  0000 L CNN
+F 0 "C50" H 3465 3646 50  0000 L CNN
 F 1 "2.2uF" H 3465 3555 50  0000 L CNN
 F 2 "Capacitor_SMD:C_1210_3225Metric_Pad1.42x2.65mm_HandSolder" H 3388 3450 50  0001 C CNN
@@
 AR Path="/5F4EF580/5F54C416/5F52D309" Ref="C12"  Part="1"
 AR Path="/5F4EF580/5F69D9D1/5F52D309" Ref="C49"  Part="1"
-F 0 "C2" H 3015 3646 50  0000 L CNN
+F 0 "C49" H 3015 3646 50  0000 L CNN
 F 1 "2.2uF" H 3015 3555 50  0000 L CNN
 F 2 "Capacitor_SMD:C_1210_3225Metric_Pad1.42x2.65mm_HandSolder" H 2938 3450 50  0001 C CNN
@@
 AR Path="/5F4EF580/5F54C416/5F52D313" Ref="C11"  Part="1"
 AR Path="/5F4EF580/5F69D9D1/5F52D313" Ref="C48"  Part="1"
-F 0 "C1" H 2565 3646 50  0000 L CNN
+F 0 "C48" H 2565 3646 50  0000 L CNN
 F 1 "2.2uF" H 2565 3555 50  0000 L CNN
 F 2 "Capacitor_SMD:C_1210_3225Metric_Pad1.42x2.65mm_HandSolder" H 2488 3450 50  0001 C CNN
@@
 AR Path="/5F4EF580/5F54C416/5F533CA4" Ref="R7"  Part="1"
 AR Path="/5F4EF580/5F69D9D1/5F533CA4" Ref="R22"  Part="1"
-F 0 "R1" H 4395 3621 50  0000 L CNN
+F 0 "R22" H 4395 3621 50  0000 L CNN
 F 1 "R" H 4395 3530 50  0000 L CNN
 F 2 "Resistor_SMD:R_0603_1608Metric_Pad1.05x0.95mm_HandSolder" V 4255 3575 50  0001 C CNN
@@
 AR Path="/5F4EF580/5F54C416/5F534F40" Ref="R8"  Part="1"
 AR Path="/5F4EF580/5F69D9D1/5F534F40" Ref="R23"  Part="1"
-F 0 "R2" H 4395 4021 50  0000 L CNN
+F 0 "R23" H 4395 4021 50  0000 L CNN
 F 1 "R" H 4395 3930 50  0000 L CNN
 F 2 "Resistor_SMD:R_0603_1608Metric_Pad1.05x0.95mm_HandSolder" V 4255 3975 50  0001 C CNN
