File: FlatSatHub.sch (KiCad schematic (older format))
At the start: 15 parts, among them J1 Jack-DC, SW1 SW_DIP_x02, SW10 SW_SPST

Commit message: V1.0 (#1)
* New layout with FPGA

- Added FPGA to ease UART and SPI signals routing
- Cleaned layout using start and circle patterns for remaining signals
- Replaced DCDC modules with better TI components

Missing stuff:
- per module PSU switch
- spare FPGA IOs connector?
- silk screen
- ...

Signed-off-by: Alexis Jeandet <alexis.jeandet@member.fsf.org>

* Most PSB done, needs more silk screen cosmetic plus review

Signed-off-by: Alexis Jeandet <alexis.jeandet@member.fsf.org>

* added some text, moved headers, added X logo, fixed res/diode overlap, fixed DRC

* Last few silk screen cleanups

Signed-off-by: Alexis Jeandet <alexis.jeandet@member.fsf.org>

Co-authored-by: pwnOrbitals <c.de-claverie@pm.me>
Parts:
- removed C1: CINCON-SIPSMT10-12, FlatSatHub:CINCON-SIPSMT10-12, symbol FlatSatHub:CINCON-SIPSMT10-12
- removed C2: bel-xRBA-06E2Ax, FlatSatHub:BEL-xRBA-06E2Ax, symbol FlatSatHub:bel-xRBA-06E2Ax
- removed D1, D2, D3: LED, LED_SMD:LED_0603_1608Metric_Pad1.05x0.95mm_HandSolder, symbol Device:LED
- removed R1, R2, R3: R, Resistor_SMD:R_0603_1608Metric_Pad1.05x0.95mm_HandSolder, symbol Device:R
- removed SW1: SW_DIP_x02, Button_Switch_THT:SW_DIP_SPSTx02_Slide_6.7x6.64mm_W7.62mm_P2.54mm_LowProfile, symbol Switch:SW_DIP_x02
- removed SW10: SW_SPST, Button_Switch_THT:SW_DIP_SPSTx01_Slide_9.78x4.72mm_W7.62mm_P2.54mm, symbol Switch:SW_SPST
Connections:
- net Vin renamed VBAT
- no-connect marks 3 -> 0
Other:
- note added: "5V -> 3A minimum\n3.3V -> 3A minimum"
- note removed: "Connector assemblies"
- note removed: "Module"
- note removed: "OBC"
- moved on the sheet: H1, H2, H3, H4, J1
