File: obc.sch (KiCad schematic (older format))
At the start: 3 parts, among them J1 DB26_Male_HighDensity_Mountin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, SW3 SW_DIP_x03

Commit message: new UART layout and rewire
Parts:
- removed J?: HEADER_4x2, symbol w_connectors:HEADER_4x2
Connections:
- net UART1_RX is gone; now on net OBC_UART1_RX: J1.23
- net UART1_TX is gone; now on net OBC_UART1_TX: J1.15
- net UART2_RX is gone; now on net OBC_UART2_RX: J1.6
- net UART2_TX is gone; now on net OBC_UART2_TX: J1.24
Changed lines of the file:
@@
 $Descr A4 11693 8268
 encoding utf-8
-Sheet 2 9
+Sheet 9 9
 Title ""
 Date ""
@@
 AR Path="/5F237C19/5F14DCB5" Ref="J16"  Part="1"
 AR Path="/5F2C117D/5F14DCB5" Ref="J?"  Part="1"
-F 0 "J4" H 5425 6217 50  0000 C CNN
+F 0 "J?" H 5425 6217 50  0000 C CNN
 F 1 "DB26_Male_HighDensity_MountingHoles" H 5425 6126 50  0000 C CNN
 F 2 "DB-HD-26:DSUB-26-HD_Male_Horizontal_P2.29x1.98mm_EdgePinOffset8.35mm_Housed_MountingHolesOffset10.89mm" H 4475 5000 50  0001 C CNN
@@
 Wire Wire Line
 	5125 5000 4725 5000
-Text Label 4725 3900 2    50   ~ 0
-UART2_RX
-Text Label 6125 3900 0    50   ~ 0
-UART2_TX
-Text Label 4725 4000 2    50   ~ 0
-UART1_TX
-Text Label 6125 4100 0    50   ~ 0
-UART1_RX
 Wire Wire Line
 	5125 3400 4525 3400
@@
 AR Path="/5F237C19/5F4B7169" Ref="#PWR0123"  Part="1"
 AR Path="/5F2C117D/5F4B7169" Ref="#PWR?"  Part="1"
-F 0 "#PWR0105" H 4525 3150 50  0001 C CNN
+F 0 "#PWR?" H 4525 3150 50  0001 C CNN
 F 1 "GND" H 4530 3227 50  0000 C CNN
 F 2 "" H 4525 3400 50  0001 C CNN
@@
 AR Path="/5F237C19/5F4B88F0" Ref="#PWR0124"  Part="1"
 AR Path="/5F2C117D/5F4B88F0" Ref="#PWR?"  Part="1"
-F 0 "#PWR0106" H 5425 5050 50  0001 C CNN
+F 0 "#PWR?" H 5425 5050 50  0001 C CNN
 F 1 "GND" H 5430 5127 50  0000 C CNN
 F 2 "" H 5425 5300 50  0001 C CNN
@@
 AR Path="/5F237C19/5F14E492" Ref="SW9"  Part="1"
 AR Path="/5F2C117D/5F14E492" Ref="SW?"  Part="1"
-F 0 "SW3" H 2975 4042 50  0000 C CNN
+F 0 "SW?" H 2975 4042 50  0000 C CNN
 F 1 "SW_DIP_x03" H 2975 3951 50  0000 C CNN
 F 2 "Button_Switch_THT:SW_DIP_SPSTx03_Slide_9.78x9.8mm_W7.62mm_P2.54mm" H 2975 3575 50  0001 C CNN
@@
 Text GLabel 2675 3575 0    50   Input ~ 0
 5V
-$Comp
-L w_connectors:HEADER_4x2 J?
-U 1 1 5F2F755E
-P 2950 4500
-F 0 "J?" H 2950 4887 60  0000 C CNN
-F 1 "HEADER_4x2" H 2950 4781 60  0000 C CNN
-F 2 "" H 2950 4500 60  0000 C CNN
-F 3 "" H 2950 4500 60  0000 C CNN
-	1    2950 4500
-	1    0    0    -1
-$EndComp
-Wire Wire Line
-	2800 4350 2500 4350
-Wire Wire Line
-	2800 4450 2500 4450
-Wire Wire Line
-	2800 4550 2500 4550
-Wire Wire Line
-	2800 4650 2500 4650
-Text Label 2500 4350 2    50   ~ 0
-UART1_RX
-Text Label 2500 4450 2    50   ~ 0
-UART1_TX
-Text Label 2500 4550 2    50   ~ 0
-UART2_RX
-Text Label 2500 4650 2    50   ~ 0
-UART2_TX
-Wire Wire Line
-	3400 4350 3100 4350
-Wire Wire Line
-	3400 4450 3100 4450
-Wire Wire Line
-	3400 4550 3100 4550
-Wire Wire Line
-	3400 4650 3100 4650
-Text GLabel 3400 4350 2    50   Input ~ 0
+Text GLabel 4725 3900 0    50   Input ~ 0
+OBC_UART2_RX
+Text GLabel 4725 4000 0    50   Input ~ 0
 OBC_UART1_TX
-Text GLabel 3400 4450 2    50   Input ~ 0
+Text GLabel 6125 3900 2    50   Input ~ 0
+OBC_UART2_TX
+Text GLabel 6125 4100 2    50   Input ~ 0
 OBC_UART1_RX
-Text GLabel 3400 4550 2    50   Input ~ 0
-OBC_UART2_TX
-Text GLabel 3400 4650 2    50   Input ~ 0
-OBC_UART2_RX
 $EndSCHEMATC

Commit message: Switch to female footprints and update positionning
Parts:
- J1: footprint DB-HD-26:DSUB-26-HD_Male_Horizontal_P2.29x1.98mm_EdgePinOffset8.35mm_Housed_MountingHolesOffset10.89mm -> Connector_Dsub:DSUB-26-HD_Female_Horizontal_P2.29x1.98mm_EdgePinOffset3.03mm_Housed_MountingHolesOffset4.94mm
Changed lines of the file:
@@
 F 0 "J15" H 5425 6217 50  0000 C CNN
 F 1 "DB26_Male_HighDensity_MountingHoles" H 5425 6126 50  0000 C CNN
-F 2 "DB-HD-26:DSUB-26-HD_Male_Horizontal_P2.29x1.98mm_EdgePinOffset8.35mm_Housed_MountingHolesOffset10.89mm" H 4475 5000 50  0001 C CNN
+F 2 "Connector_Dsub:DSUB-26-HD_Female_Horizontal_P2.29x1.98mm_EdgePinOffset3.03mm_Housed_MountingHolesOffset4.94mm" H 4475 5000 50  0001 C CNN
 F 3 "https://www.mouser.fr/ProductDetail/Kycon/K66X-A26S-N?qs=C%252BuF95oynlmx3ziDhlO2Bg%3D%3D" H 4475 5000 50  0001 C CNN
 	1    5425 4600

Commit message: V1.0 (#1)
* New layout with FPGA

- Added FPGA to ease UART and SPI signals routing
- Cleaned layout using start and circle patterns for remaining signals
- Replaced DCDC modules with better TI components

Missing stuff:
- per module PSU switch
- spare FPGA IOs connector?
- silk screen
- ...

Signed-off-by: Alexis Jeandet <alexis.jeandet@member.fsf.org>

* Most PSB done, needs more silk screen cosmetic plus review

Signed-off-by: Alexis Jeandet <alexis.jeandet@member.fsf.org>

* added some text, moved headers, added X logo, fixed res/diode overlap, fixed DRC

* Last few silk screen cleanups

Signed-off-by: Alexis Jeandet <alexis.jeandet@member.fsf.org>

Co-authored-by: pwnOrbitals <c.de-claverie@pm.me>
Parts:
- removed SW3: SW_DIP_x03, Button_Switch_THT:SW_DIP_SPSTx03_Slide_9.78x9.8mm_W7.62mm_P2.54mm, symbol Switch:SW_DIP_x03
Changed lines of the file:
@@
 $Descr A4 11693 8268
 encoding utf-8
-Sheet 9 9
+Sheet 9 13
 Title ""
 Date ""
@@
 	1    0    0    -1
 $EndComp
-$Comp
-L Switch:SW_DIP_x03 SW3
-U 1 1 5F2D876D
-P 2975 3575
-AR Path="/5F1123F9/5F10EEE2/5F2D876D" Ref="SW3"  Part="1"
-AR Path="/5F11264C/5F10EEE2/5F2D876D" Ref="SW4"  Part="1"
-AR Path="/5F10DACE/5F10EEE2/5F2D876D" Ref="SW2"  Part="1"
-AR Path="/5F11264F/5F10EEE2/5F2D876D" Ref="SW5"  Part="1"
-AR Path="/5F11285A/5F10EEE2/5F2D876D" Ref="SW6"  Part="1"
-AR Path="/5F11285D/5F10EEE2/5F2D876D" Ref="SW7"  Part="1"
-AR Path="/5F112860/5F10EEE2/5F2D876D" Ref="SW8"  Part="1"
-AR Path="/5F112863/5F10EEE2/5F2D876D" Ref="SW9"  Part="1"
-AR Path="/5F1F8EB1/5F2D876D" Ref="SW2"  Part="1"
-AR Path="/5F202513/5F2D876D" Ref="SW?"  Part="1"
-AR Path="/5F214496/5F2D876D" Ref="SW?"  Part="1"
-AR Path="/5F2144C2/5F2D876D" Ref="SW?"  Part="1"
-AR Path="/5F21C578/5F2D876D" Ref="SW?"  Part="1"
-AR Path="/5F21C5A4/5F2D876D" Ref="SW?"  Part="1"
-AR Path="/5F21C5D0/5F2D876D" Ref="SW?"  Part="1"
-AR Path="/5F21C5FC/5F2D876D" Ref="SW?"  Part="1"
-AR Path="/5F22A1CE/5F2D876D" Ref="SW3"  Part="1"
-AR Path="/5F22D207/5F2D876D" Ref="SW4"  Part="1"
-AR Path="/5F22D233/5F2D876D" Ref="SW5"  Part="1"
-AR Path="/5F2317AE/5F2D876D" Ref="SW6"  Part="1"
-AR Path="/5F2317DA/5F2D876D" Ref="SW7"  Part="1"
-AR Path="/5F237BED/5F2D876D" Ref="SW8"  Part="1"
-AR Path="/5F237C19/5F2D876D" Ref="SW9"  Part="1"
-AR Path="/5F2C117D/5F2D876D" Ref="SW2"  Part="1"
-F 0 "SW2" H 2975 4042 50  0000 C CNN
-F 1 "SW_DIP_x03" H 2975 3951 50  0000 C CNN
-F 2 "Button_Switch_THT:SW_DIP_SPSTx03_Slide_9.78x9.8mm_W7.62mm_P2.54mm" H 2975 3575 50  0001 C CNN
-F 3 "~" H 2975 3575 50  0001 C CNN
-	1    2975 3575
-	1    0    0    -1
-$EndComp
